Commit message: Got the pendulum working as well as a model for the franka panda that is editable - need to get the propper EE model

File: src/simulation/models/strawberry_cluster.urdf (robot description, URDF)
Before this commit: robot strawberry_plant, 4 links, 3 joints
Links:
- link Upperstem: mass 1. -> None; geometry visual sphere radius=0.01
- link stem: mass 100 -> 0.01; geometry collision cylinder length=0.1 radius=0.001; visual cylinder length=0.1 radius=0.001
- link strawberry: mass 500 -> 0.04
Joints:
- joint joint0: origin (none) -> xyz=0 0 0 rpy=0 0 0; type continuous -> fixed
- joint joint1: axis 1 1 0 -> (none); origin xyz=0 0 0 rpy=0 0 0 -> xyz=0 0 0 rpy=0 0 0.75
- joint joint2: origin (none) -> xyz=0 0 0 rpy=0 0 0
